File: control/quantizer_control.sch (EAGLE design)
At the start: 111 parts, among them IC1 74HC595D, IC2 74HC595D

Commit message: SAD
Parts:
- removed AGND, AGND6, AGND7, AGND8, CLKOUT, DAT1, DAT2, GND, GND5, GND6, GND7, IN1, IN2, IN3, IN4, IN5, IN6, JP1, JP22, JP23, JP24, JP25, MIDIR, MIDIT, OUT1, OUT2, OUT3, OUT4, POT, RCK, SCK, VCC, VREF: (no value), pinhead:PINHD-1X1
- removed CKOUT, CVIN1, CVIN2, CVIN3, CVIN4, CVIN5, CVIN6, CVOUT1, CVOUT2, CVOUT3, CVOUT4: WQP-PJ301M-12_JACK, thonkiconn:WQP-PJ301M-12_JACK
- removed IC1, IC2: 74HC595D, 74xx-eu:74HC595D
- removed LED10, LED11, LED12, LED3, LED4, LED5, LED6, LED7, LED8, LED9: (no value), led:LED3MM
- removed MIDI_IN: VERTICAL_3_5MM_SOCKETTHONK, jason_eagle6:VERTICAL_3_5MM_SOCKETTHONK
- removed R10, R11, R12, R3, R4, R5, R6, R7, R8, R9: (no value), rcl:R-EU_R0805
- removed S1, S10, S11, S12, S13, S14, S15, S16, S17, S18, S2, S3, S4, S5, S6, S7, S8, S9: (no value), switch-omron:10-XX
- removed U$12, U$28, U$29, U$30: 0805DIODE, jasons_stuff:0805DIODE
- added C4, C5, C6, C7, C8, C9: (no value), rcl:C-EUC0805
- added D1, D10, D11, D12, D13, D14, D15, D16, D17, D2, D3, D4, D5, D6, D7, D8, D9: 0805DIODE, jasons_stuff:0805DIODE
- added SW1, SW10, SW11, SW12, SW13, SW14, SW15, SW16, SW17, SW18, SW2, SW3, SW4, SW5, SW6, SW7, SW8, SW9: SKPMSWITCH, jason_eagle6:SKPMSWITCH
- added U$1: 2X8SMT, jason_eagle6:2X8SMT
- added U$10, U$11, U$2, U$3, U$4, U$5, U$6, U$7, U$8, U$9: APA102-2020, jason_eagle6:APA102-2020
- LED1, LED2: device led:LED3MM -> led:LEDCHIP-LED0805
- U$13: value ALPS_POT_SMALL -> APA102-2020; device jasons_stuff:ALPS_POT_SMALL -> jason_eagle6:APA102-2020
- U$14, U$15, U$16, U$17, U$18, U$19, U$20, U$21, U$22, U$23, U$24, U$25, U$26, U$27: value 0805DIODE -> APA102-2020; device jasons_stuff:0805DIODE -> jason_eagle6:APA102-2020
Connections:
- removed net AGND: AGND.1, AGND6.1, AGND7.1, AGND8.1, C1.2, CKOUT.1, CVIN1.1, CVIN1.3, CVIN2.1, CVIN2.3, CVIN3.1, CVIN3.3, CVIN4.1, CVIN4.3, CVIN5.1, CVIN5.3, CVIN6.1, CVIN6.3, CVOUT1.1, CVOUT2.1, CVOUT3.1, CVOUT4.1, U$13.A
- removed net N$66: IC1A.RCK, IC2A.RCK, RCK.1
- removed net N$67: IC1A.SCK, IC2A.SCK, SCK.1
- removed net N$68: DAT1.1, IC1A.SER
- removed net N$69: DAT2.1, IC2A.SER
- removed net VREF: U$13.B, VREF.1
- new net ALED_MOSI: U$1.15, U$2.SDI
- new net ALED_SCK: U$1.16, U$2.CKI
- new net CKI2: U$14.CKO, U$15.CKI
- new net COM0: SW1.2, SW2.2, SW3.2, SW4.2, SW5.2, SW6.2, U$1.6
- new net COM1: SW10.2, SW11.2, SW12.2, SW7.2, SW8.2, SW9.2, U$1.4
- new net COM2: SW13.2, SW14.2, SW15.2, SW16.2, SW17.2, U$1.13
- new net KEY0: D1.P$1, D12.P$1, D15.P$1, U$1.8
- new net KEY1: D11.P$1, D16.P$1, D2.P$1, U$1.10
- new net KEY2: D10.P$1, D17.P$1, D3.P$1, U$1.12
- new net KEY3: D13.P$1, D4.P$1, D9.P$1, U$1.3
- new net KEY4: D14.P$1, D5.P$1, D8.P$1, U$1.5
- new net KEY5: D6.P$1, D7.P$1, U$1.7
- new net LED0: R1.2, U$1.9
- new net LED1: R2.2, U$1.11
- new net N$62: D16.P$2, SW14.1
- new net N$63: D17.P$2, SW15.1
- new net N$64: D13.P$2, SW16.1
- new net N$65: D14.P$2, SW17.1
- new net SDI2: U$14.SDO, U$15.SDI
- new net SW1: SW18.1, U$1.14
- net GND: now also C1.2, C2.2, C3.2, C4.2, C5.2, C6.2, C7.2, C8.2, C9.2, LED1.C, LED2.C, SW18.2, U$1.1, U$10.GND, U$11.GND, U$13.GND, U$14.GND, U$15.GND, U$16.GND, U$17.GND, U$18.GND, U$19.GND, U$2.GND, U$20.GND, U$21.GND, U$22.GND, U$23.GND, U$24.GND, U$25.GND, U$26.GND, U$27.GND, U$3.GND, U$4.GND, U$5.GND, U$6.GND, U$7.GND, U$8.GND, U$9.GND; no longer C2.1, C3.1, GND.1, GND5.1, GND6.1, GND7.1, IC1A.G, IC1P.GND, IC2A.G, IC2P.GND
- net N$1: now also U$26.SDO, U$27.SDI; no longer IC1A.QA, LED1.A, U$12.P$2
- net N$10: now also D6.P$2, SW6.1; no longer IC2A.QC, LED10.A, U$22.P$2, U$28.P$2
- net N$11: now also U$3.SDO, U$4.SDI; no longer IC2A.QB, LED11.A, U$23.P$2, U$29.P$2
- net N$12: now also U$3.CKO, U$4.CKI; no longer IC2A.QA, LED12.A, U$24.P$2, U$30.P$2
- net N$13: now also U$4.SDO, U$5.SDI; no longer LED1.C, R1.1
- net N$14: now also U$4.CKO, U$5.CKI; no longer LED2.C, R2.1
- net N$15: now also U$5.SDO, U$6.SDI; no longer LED3.C, R3.1
- net N$16: now also U$5.CKO, U$6.CKI; no longer LED4.C, R4.1
- net N$17: now also U$6.SDO, U$7.SDI; no longer LED5.C, R5.1
- net N$18: now also U$6.CKO, U$7.CKI; no longer LED6.C, R6.1
- net N$19: now also U$7.SDO, U$8.SDI; no longer LED7.C, R7.1
- net N$2: now also U$26.CKO, U$27.CKI; no longer IC1A.QB, LED2.A, U$14.P$2
- net N$20: now also U$7.CKO, U$8.CKI; no longer LED8.C, R8.1
- net N$21: now also U$8.SDO, U$9.SDI; no longer LED9.C, R9.1
- net N$22: now also U$8.CKO, U$9.CKI; no longer LED10.C, R10.1
- net N$23: now also U$10.SDI, U$9.SDO; no longer LED11.C, R11.1
- net N$24: now also U$10.CKI, U$9.CKO; no longer LED12.C, R12.1
- net N$25: now also U$10.SDO, U$11.SDI; no longer JP24.1, R1.2, R2.2, R3.2, R4.2, R5.2, R6.2
- net N$26: now also U$10.CKO, U$11.CKI; no longer JP23.1, R10.2, R11.2, R12.2, R7.2, R8.2, R9.2
- net N$27: now also U$11.SDO, U$13.SDI; no longer S6.P, U$18.P$1
- net N$28: now also U$11.CKO, U$13.CKI; no longer S5.P, U$17.P$1
- net N$29: now also U$13.SDO, U$14.SDI; no longer S4.P, U$16.P$1
- net N$3: now also D1.P$2, SW1.1; no longer IC1A.QC, LED3.A, U$15.P$2
- net N$30: now also D7.P$2, SW7.1; no longer S3.P, U$15.P$1
- net N$31: now also U$13.CKO, U$14.CKI; no longer S2.P, U$14.P$1
- net N$32: now also LED1.A, R1.1; no longer S1.P, U$12.P$1
- net N$33: now also U$15.SDO, U$16.SDI; no longer JP22.1, S1.S, S2.S, S3.S, S4.S, S5.S, S6.S
- net N$34: now also U$15.CKO, U$16.CKI; no longer S12.P, U$24.P$1
- net N$35: now also U$16.SDO, U$17.SDI; no longer S11.P, U$23.P$1
- net N$36: now also D8.P$2, SW8.1; no longer S10.P, U$22.P$1
- net N$37: now also U$16.CKO, U$17.CKI; no longer S9.P, U$21.P$1
- net N$38: now also U$17.SDO, U$18.SDI; no longer S8.P, U$20.P$1
- net N$39: now also U$17.CKO, U$18.CKI; no longer S7.P, U$19.P$1
- net N$4: now also D2.P$2, SW2.1; no longer IC1A.QD, LED4.A, U$16.P$2
- net N$40: now also U$18.SDO, U$19.SDI; no longer JP25.1, S10.S, S11.S, S12.S, S7.S, S8.S, S9.S
- net N$41: now also U$18.CKO, U$19.CKI; no longer S13.P, U$30.P$1
- net N$42: now also U$19.SDO, U$20.SDI; no longer S14.P, U$29.P$1
- net N$43: now also U$19.CKO, U$20.CKI; no longer S15.P, U$28.P$1
- net N$44: now also U$20.SDO, U$21.SDI; no longer S16.P, U$27.P$1
- net N$45: now also D9.P$2, SW9.1; no longer S17.P, U$26.P$1
- net N$46: now also U$20.CKO, U$21.CKI; no longer S18.P, U$25.P$1
- net N$47: now also U$21.SDO, U$22.SDI; no longer JP1.1, S13.S, S14.S, S15.S, S16.S, S17.S, S18.S
- net N$48: now also U$21.CKO, U$22.CKI; no longer MIDIT.1, MIDI_IN.4
- net N$49: now also D10.P$2, SW10.1; no longer CVIN6.2, IN6.1
- net N$5: now also D3.P$2, SW3.1; no longer IC1A.QE, LED5.A, U$17.P$2
- net N$50: now also U$22.SDO, U$23.SDI; no longer CVIN5.2, IN5.1
- net N$51: now also U$22.CKO, U$23.CKI; no longer CVIN4.2, IN4.1
- net N$52: now also U$23.SDO, U$24.SDI; no longer CVOUT3.2, OUT3.1
- net N$53: now also U$23.CKO, U$24.CKI; no longer CVOUT2.2, OUT2.1
- net N$54: now also U$24.SDO, U$25.SDI; no longer CVIN3.2, IN3.1
- net N$55: now also U$24.CKO, U$25.CKI; no longer CVIN2.2, IN2.1
- net N$56: now also U$25.SDO, U$26.SDI; no longer CVIN1.2, IN1.1
- net N$57: now also U$25.CKO, U$26.CKI; no longer CVOUT1.2, OUT1.1
- net N$58: now also LED2.A, R2.1; no longer CKOUT.2, CLKOUT.1
- net N$59: now also D11.P$2, SW11.1; no longer CVOUT4.2, OUT4.1
- net N$6: now also D4.P$2, SW4.1; no longer IC1A.QF, LED6.A, U$18.P$2
- net N$60: now also D12.P$2, SW12.1; no longer MIDIR.1, MIDI_IN.3
- net N$61: now also D15.P$2, SW13.1; no longer C1.1, POT.1, U$13.W
- net N$7: now also D5.P$2, SW5.1; no longer IC2A.QF, LED7.A, U$19.P$2, U$25.P$2
- net N$8: now also U$2.SDO, U$3.SDI; no longer IC2A.QE, LED8.A, U$20.P$2, U$26.P$2
- net N$9: now also U$2.CKO, U$3.CKI; no longer IC2A.QD, LED9.A, U$21.P$2, U$27.P$2
- net VCC: now also C1.1, C2.1, C3.1, C4.1, C5.1, C6.1, C7.1, C8.1, C9.1, U$1.2, U$10.VCC, U$11.VCC, U$13.VCC, U$14.VCC, U$15.VCC, U$16.VCC, U$17.VCC, U$18.VCC, U$19.VCC, U$2.VCC, U$20.VCC, U$21.VCC, U$22.VCC, U$23.VCC, U$24.VCC, U$25.VCC, U$26.VCC, U$27.VCC, U$3.VCC, U$4.VCC, U$5.VCC, U$6.VCC, U$7.VCC, U$8.VCC, U$9.VCC; no longer C2.2, C3.2, IC1A.SCL, IC1P.VCC, IC2A.SCL, IC2P.VCC, VCC.1
Other:
- moved on the sheet: C1, C2, C3, LED1, LED2, R1, R2
