File: main/quantizer_main.brd (EAGLE design)
At the start: 108 x 40 mm, 141 parts, among them IC1 TL074D, IC100 REG1117, IC2 TL074D, IC200 REG1117, IC3 TL074D, IC3000 6N138, IC4 TL074D, IC500 MAX6070, IC600 MAX1303_ADC, IC700 MAX5134_DAC, IC800 MKE02_44PIN

Commit message: ewr
Parts:
- moved TP6 82.4 mm to (58.1, 6.35)
- moved TP5 71.0 mm to (56.1, 15.4)
- moved TP3 55.8 mm to (64.2, 32.1)
- moved TP7 55.1 mm to (21.7, 23.4)
- moved TP4 51.1 mm to (64.6, 43.2)
- moved TP1 47.2 mm to (54.5, 31.9)
- moved TP2 38.5 mm to (54.2, 43.2)
- moved R1601 1.27 mm to (60.7, 6.86)
Connections:
- net CVIN0: now also TP1.TP
- net CVIN1: now also TP2.TP
- net CVIN2: now also TP3.TP
- net CVIN3: now also TP4.TP
- net CVIN5: now also TP5.TP
- net CVIN6: now also TP6.TP
- net CVIN7: now also TP7.TP
Routing:
- net CVIN7: track 31.8 -> 36.2 mm
- net CVIN0: track 18.8 -> 21.1 mm
- net CVIN3: track 9.09 -> 11.1 mm
- net CVIN1: track 14.3 -> 16.2 mm
- net -12V: track 186.5 -> 184.7 mm
- net CVIN2: track 8.93 -> 10.6 mm
- net CVIN5: track 46.3 -> 47.8 mm
- net CVIN6: track 2.76 -> 4.03 mm
- net AGND: vias 18 -> 17

Commit message: sddd
Parts:
- removed TP9: TPB1,27, testpad:B1,27
Connections:
- net N$50 renamed OFFSET
- removed net N$46: IC800.15, TP9.TP
- net CVIN6: now also IC800.15
Routing:
- net CVIN6: track 4.03 -> 45.5 mm, vias 0 -> 2
- net N$46: track 3.47 -> 0.00 mm
- net +12V: track 244.4 -> 246.6 mm
- net DAC_READY: track 92.5 -> 91.3 mm
- net GND: track 42.7 -> 43.8 mm, vias 8 -> 11

Commit message: sf
Parts:
- removed C1401, C802: (no value), rcl:C0805
- removed IC600: MAX1303_ADC, jason_eagle6:TSSOP20
- removed TP10: TPB1,27, testpad:B1,27
- added C29, C30: (no value), rcl:E2-5
- added IC6: TL074D, linear:SO14
- added PD7: TPB1,27, testpad:B1,27
- C19, C20: device rcl:E2-5 -> rcl:C0805
- IC3: value TL074D -> MAX1303_ADC; device linear:SO14 -> jason_eagle6:TSSOP20
- moved IC1 45.0 mm to (96.3, 38.6)
- moved IC3 36.8 mm to (59.4, 37.6)
- moved C20 35.3 mm to (46.9, 10.5), flipped to the bottom, turned to 180 degrees
- moved C19 29.8 mm to (43.9, 20.7), flipped to the bottom, turned to 270 degrees
- moved IC4 27.5 mm to (51.3, 37.6)
- renumbered C100 to C15, C1000 to C12, C1001 to C13, C101 to C14, C102 to C32, C1200 to C8, C1201 to C7, C1400 to C23, C1500 to C22, C1700 to C16, C200 to C35, C2000 to C1, C2001 to C3, C2002 to C5, C201 to C34, C202 to C31, C203 to C33, C2100 to C2, C2200 to C6, C2300 to C4, C2400 to C21, C500 to C27, C501 to C28, C600 to C10, C601 to C9, C603 to C11, C700 to C24, C701 to C26, C702 to C25, C800 to C17, C801 to C18, CVINA to IN2, CVINB to IN1, CVINC to IN5, CVIND to IN4, CVINE to IN3, CVINF to IN6, CVOUTA to OUT4, CVOUTB to OUT3, CVOUTC to OUT1, CVOUTD to OUT2, D3000 to D3, FB1 to L1, FB2 to L2, IC100 to IC9, IC200 to IC10, IC3000 to IC11, IC500 to IC8, IC700 to IC7, IC800 to IC5, JP1 to PWR, JP23 to ICSP, MIDIIN to MIDI, PTC1 to F1, PTC2 to F2, R1000 to R28, R1001 to R26, R1002 to R22, R1003 to R27, R1100 to R25, R1101 to R23, R1102 to R21, R1103 to R24, R1200 to R16, R1201 to R18, R1202 to R20, R1203 to R17, R1300 to R13, R1301 to R15, R1302 to R14, R1303 to R19, R1400 to R33, R1401 to R34, R1500 to R41, R1501 to R40, R1600 to R35, R1601 to R36, R2000 to R1, R2001 to R2, R2002 to R3, R2100 to R4, R2101 to R5, R2102 to R6, R2200 to R12, R2201 to R11, R2202 to R10, R2300 to R9, R2301 to R8, R2302 to R7, R2400 to R39, R2401 to R38, R2402 to R37, R3000 to R29, R3001 to R30, R3002 to R32, R3003 to R31, R3004 to R42, R3005 to R43, R4000 to R44, TP1 to A, TP11 to PD6, TP12 to PD5, TP13 to PB4, TP2 to B, TP3 to C, TP4 to D, TP5 to E, TP6 to F, TP7 to G, TP8 to PB5, TRGOUT to TRIG, U$14 to POT1
Connections:
- removed net CVIN7: C16.1, G.TP, IC5.19, POT1.W
- new net CVIN4: E.TP, IC5.14, IC6.1, R34.2
- net +12V: now also C29.+, IC6.4; no longer C19.+, IC3.4
- net +5V: now also IC3.16, IC3.19, IC3.2; no longer IC600.16, IC600.19, IC600.2
- net -12V: now also C20.2, C30.-, IC6.11; no longer C1401.2, C20.-, IC3.11
- net 4.096V: now also IC3.17; no longer IC600.17
- net ADC_CSEL: now also IC3.7; no longer IC600.7
- net ADC_SSTRB: now also IC3.9; no longer IC600.9
- net AGND: now also C20.1, C29.-, C30.+, IC3.1, IC3.18, IC3.20, IC4.10, IC4.12, IC4.3, IC4.5; no longer C1401.1, C19.-, C20.+, IC1.10, IC1.12, IC1.3, IC1.5, IC600.1, IC600.18, IC600.20
- net CVIN0: now also IC3.4, IC4.7; no longer IC1.7, IC600.4
- net CVIN1: now also IC3.3, IC4.1; no longer IC1.1, IC600.3
- net CVIN2: now also IC3.6; no longer IC600.6
- net CVIN3: now also IC3.5; no longer IC600.5
- net CVIN5: now also F.TP, IC5.15, IC6.7, R36.2; no longer E.TP, IC4.1, IC5.14, R34.2
- net CVIN6: now also C16.1, G.TP, IC5.19, POT1.W; no longer F.TP, IC4.7, IC5.15, R36.2
- net CVOUTA: now also IC1.3; no longer IC3.3
- net CVOUTB: now also IC1.5; no longer IC3.5
- net CVOUTC: now also IC1.10; no longer IC3.10
- net CVOUTD: now also IC1.12; no longer IC3.12
- net GND: now also C19.2, IC3.12, IC3.13; no longer C802.2, IC600.12, IC600.13
- net N$1: now also IC1.2; no longer IC3.2
- net N$11: now also IC1.9; no longer IC3.9
- net N$13: now also IC1.8; no longer IC3.8
- net N$15: now also IC4.9; no longer IC1.9
- net N$16: now also IC1.13; no longer IC3.13
- net N$18: now also IC1.14; no longer IC3.14
- net N$20: now also IC4.8; no longer IC1.8
- net N$21: now also IC4.6; no longer IC1.6
- net N$25: now also IC4.13; no longer IC1.13
- net N$26: now also IC4.14; no longer IC1.14
- net N$27: now also IC4.2; no longer IC1.2
- net N$34: now also IC6.13; no longer IC4.13
- net N$35: now also IC6.14; no longer IC4.14
- net N$4: now also IC1.1; no longer IC3.1
- net N$42: now also IC6.10; no longer IC4.10
- net N$43: now also IC6.2; no longer IC4.2
- net N$47: now also IC6.6; no longer IC4.6
- net N$48: now also PD7.TP; no longer TP10.TP
- net N$6: now also IC1.6; no longer IC3.6
- net N$8: now also IC1.7; no longer IC3.7
- net OFFSET: now also IC6.3, IC6.5, IC6.8, IC6.9; no longer IC4.3, IC4.5, IC4.8, IC4.9
- net SPI_CLK: now also IC3.10; no longer IC600.10
- net SPI_MISO: now also IC3.11; no longer IC600.11
- net SPI_MOSI: now also IC3.8; no longer IC600.8
- net TRGOUT: now also IC6.12; no longer IC4.12
- net VDD: now also C19.1, IC3.14, IC3.15; no longer C802.1, IC600.14, IC600.15
Routing:
- net CVIN4: track 0.00 -> 47.8 mm, vias 0 -> 4
- net CVIN7: track 36.2 -> 0.00 mm
- net CVIN6: track 45.5 -> 36.2 mm, vias 2 -> 0
- net CVIN5: track 47.8 -> 45.5 mm, vias 4 -> 2
- net N$48: track 4.29 -> 6.05 mm

Commit message: asd
Parts:
- moved G 6.55 mm to (15.2, 23.6)
- moved JP10 2.84 mm to (21.3, 8.13)
- moved JP9 2.84 mm to (31.5, 8.13)
- moved JP11 2.84 mm to (21.3, 10.7)
- moved JP8 2.84 mm to (31.5, 10.7)
- moved JP13 2.84 mm to (18.8, 8.13)
- moved JP14 2.84 mm to (16.3, 8.13)
- moved JP17 2.84 mm to (34.0, 8.13)
- moved JP3 2.84 mm to (23.9, 8.13)
- moved JP5 2.84 mm to (26.4, 8.13)
- moved JP7 2.84 mm to (29.0, 8.13)
- moved JP12 2.84 mm to (18.8, 10.7)
- moved JP15 2.84 mm to (16.3, 10.7)
- moved JP16 2.84 mm to (34.0, 10.7)
- moved JP2 2.84 mm to (23.9, 10.7)
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Connections:
- net AGND: now also C16.2, POT1.A
- net GND: no longer C16.2, POT1.A
Routing:
- net GND: track 43.5 -> 67.5 mm
- net AGND: track 47.1 -> 53.3 mm
- net KEY7: track 10.7 -> 16.6 mm
- net VDD: track 210.3 -> 204.8 mm
- net KEY6: track 7.82 -> 12.6 mm, vias 0 -> 1
- net CVIN6: track 36.2 -> 33.5 mm
- net KEY5: track 11.1 -> 13.5 mm
- net KEY10: track 28.3 -> 26.0 mm
- net KEY11: track 32.6 -> 30.3 mm
- net ALED_MOSI: track 23.4 -> 22.2 mm
- net KEY4: track 8.73 -> 9.93 mm, vias 0 -> 1
- net KEY1: track 13.9 -> 15.1 mm
- net KEY0: track 11.2 -> 12.2 mm
- net KEY2: track 10.3 -> 11.3 mm
- net KEY3: track 12.5 -> 13.4 mm
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
Commit message: v1 pcb?
Parts:
- added C36: (no value), resistor:C0805
- added IC12: 24LC_16BT-I/OT, Microchip-24LCxxx:SOT95P290X145-5N
- added R45, R46: (no value), rcl:R0805
Connections:
- net +5V: now also C36.2, IC12.4, R45.2, R46.2
- net GND: now also C36.1, IC12.2, IC12.5
- net SCL: now also IC12.1, R45.1
- net SDA: now also IC12.3, R46.1
Routing:
- net SDA: track 0.00 -> 42.6 mm, vias 0 -> 2
- net SCL: track 0.00 -> 40.4 mm, vias 0 -> 2
- net +5V: track 204.1 -> 218.3 mm
- net CVIN5: track 45.5 -> 49.9 mm
- net KEY10: track 26.0 -> 29.0 mm
- net ADC_CSEL: track 52.7 -> 49.7 mm
- net KEY11: track 30.3 -> 33.1 mm
- net ADC_SSTRB: track 38.6 -> 37.1 mm
- net GND: vias 11 -> 12
Other:
- board text added: "cv quantizer main v1"
- board text added: "hotchk155"
