File: main/quantizer_main.brd (EAGLE design)
At the start: 108 x 40 mm, 144 parts, among them IC1 TL074D, IC10 REG1117, IC11 6N138, IC12 24LC_16BT-I/OT, IC2 TL074D, IC3 MAX1303_ADC, IC4 TL074D, IC5 MKE02_44PIN, IC6 TL074D, IC7 MAX5134_DAC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

Commit message: c21 10n
Parts:
- C21: value (none) -> 10n
Changed lines of the file:
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@@
 <attribute name="VALUE" x="38.1" y="13.081" size="1.27" layer="28" rot="MR90"/>
 </element>
-<element name="C21" library="rcl" package="C0805" value="" x="48.26" y="13.716" smashed="yes" rot="MR270">
+<element name="C21" library="rcl" package="C0805" value="10n" x="48.26" y="13.716" smashed="yes" rot="MR270">
 <attribute name="NAME" x="48.006" y="16.9545" size="1.27" layer="26" font="vector" ratio="20" rot="MR180"/>
 <attribute name="VALUE" x="50.8" y="14.986" size="1.27" layer="28" rot="MR270"/>

Commit message: asd
Parts:
- C1, C2, C4, C6: value (none) -> 200p
- R33, R35: value (none) -> 120k
- R34, R36, R40: value (none) -> 22k
- R41: value (none) -> 100k
Connections:
- net CVIN4 renamed MCUADC3
- net CVIN5 renamed MCUADC2
- net CVIN6 renamed MCUADC1
Changed lines of the file:
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@@
 <attribute name="VALUE" x="107.95" y="41.529" size="1.27" layer="28" rot="MR90"/>
 </element>
-<element name="C1" library="rcl" package="C0805" value="" x="102.87" y="42.164" smashed="yes" rot="MR270">
+<element name="C1" library="rcl" package="C0805" value="200p" x="102.87" y="42.164" smashed="yes" rot="MR270">
 <attribute name="NAME" x="101.7905" y="43.307" size="1.27" layer="26" font="vector" ratio="20" rot="MR270"/>
 <attribute name="VALUE" x="105.41" y="43.434" size="1.27" layer="28" rot="MR270"/>
@@
 <attribute name="VALUE" x="113.03" y="35.56" size="1.27" layer="28" rot="MR270"/>
 </element>
-<element name="C2" library="rcl" package="C0805" value="" x="102.87" y="35.052" smashed="yes" rot="MR90">
+<element name="C2" library="rcl" package="C0805" value="200p" x="102.87" y="35.052" smashed="yes" rot="MR90">
 <attribute name="NAME" x="102.235" y="30.9245" size="1.27" layer="26" font="vector" ratio="20" rot="MR90"/>
 <attribute name="VALUE" x="100.33" y="33.782" size="1.27" layer="28" rot="MR90"/>
@@
 <attribute name="VALUE" x="84.582" y="35.687" size="1.27" layer="28" rot="MR270"/>
 </element>
-<element name="C6" library="rcl" package="C0805" value="" x="89.662" y="35.052" smashed="yes" rot="MR90">
+<element name="C6" library="rcl" package="C0805" value="200p" x="89.662" y="35.052" smashed="yes" rot="MR90">
 <attribute name="NAME" x="92.0115" y="36.576" size="1.27" layer="26" font="vector" ratio="20" rot="MR270"/>
 <attribute name="VALUE" x="87.122" y="33.782" size="1.27" layer="28" rot="MR90"/>
@@
 <attribute name="VALUE" x="79.502" y="41.529" size="1.27" layer="28" rot="MR90"/>
 </element>
-<element name="C4" library="rcl" package="C0805" value="" x="89.662" y="42.164" smashed="yes" rot="MR270">
+<element name="C4" library="rcl" package="C0805" value="200p" x="89.662" y="42.164" smashed="yes" rot="MR270">
 <attribute name="NAME" x="92.0115" y="43.4975" size="1.27" layer="26" font="vector" ratio="20" rot="MR270"/>
 <attribute name="VALUE" x="92.202" y="43.434" size="1.27" layer="28" rot="MR270"/>
@@
 <attribute name="NAME" x="54.8005" y="14.859" size="1.27" layer="26" font="vector" ratio="20" rot="MR0"/>
 </element>
-<element name="R33" library="rcl" package="R0805" value="" x="64.008" y="14.478" smashed="yes" rot="MR0">
+<element name="R33" library="rcl" package="R0805" value="120k" x="64.008" y="14.478" smashed="yes" rot="MR0">
 <attribute name="NAME" x="66.548" y="15.748" size="1.27" layer="26" font="vector" ratio="20" rot="MR0"/>
 <attribute name="VALUE" x="64.643" y="11.938" size="1.27" layer="28" rot="MR0"/>
 </element>
-<element name="R40" library="rcl" package="R0805" value="" x="45.72" y="7.239" smashed="yes" rot="MR90">
+<element name="R40" library="rcl" package="R0805" value="22k" x="45.72" y="7.239" smashed="yes" rot="MR90">
 <attribute name="NAME" x="41.7195" y="10.0965" size="1.27" layer="26" font="vector" ratio="20" rot="MR180"/>
 <attribute name="VALUE" x="43.18" y="6.604" size="1.27" layer="28" rot="MR90"/>
 </element>
-<element name="R41" library="rcl" package="R0805" value="" x="43.18" y="7.239" smashed="yes" rot="MR270">
+<element name="R41" library="rcl" package="R0805" value="100k" x="43.18" y="7.239" smashed="yes" rot="MR270">
 <attribute name="NAME" x="41.656" y="5.08" size="1.27" layer="26" font="vector" ratio="20" rot="MR0"/>
 <attribute name="VALUE" x="45.72" y="7.874" size="1.27" layer="28" rot="MR270"/>
 </element>
-<element name="R34" library="rcl" package="R0805" value="" x="59.436" y="14.478" smashed="yes" rot="MR0">
+<element name="R34" library="rcl" package="R0805" value="22k" x="59.436" y="14.478" smashed="yes" rot="MR0">
 <attribute name="NAME" x="61.1505" y="15.621" size="1.27" layer="26" font="vector" ratio="20" rot="MR0"/>
 <attribute name="VALUE" x="60.071" y="11.938" size="1.27" layer="28" rot="MR0"/>
@@
 <attribute name="NAME" x="81.3054" y="24.9682" size="1.27" layer="21" font="vector" ratio="20" rot="R180"/>
 </element>
-<element name="R35" library="rcl" package="R0805" value="" x="65.024" y="8.382" smashed="yes" rot="MR0">
+<element name="R35" library="rcl" package="R0805" value="120k" x="65.024" y="8.382" smashed="yes" rot="MR0">
 <attribute name="NAME" x="66.675" y="9.652" size="1.27" layer="26" font="vector" ratio="20" rot="MR0"/>
 <attribute name="VALUE" x="65.659" y="5.842" size="1.27" layer="28" rot="MR0"/>
 </element>
-<element name="R36" library="rcl" package="R0805" value="" x="60.706" y="6.858" smashed="yes" rot="MR0">
+<element name="R36" library="rcl" package="R0805" value="22k" x="60.706" y="6.858" smashed="yes" rot="MR0">
 <attribute name="NAME" x="65.9765" y="5.2705" size="1.27" layer="26" font="vector" ratio="20" rot="MR0"/>
 <attribute name="VALUE" x="61.341" y="4.318" size="1.27" layer="28" rot="MR0"/>
@@
 <wire x1="60.386" y1="13.523" x2="60.198" y2="13.335" width="0.254" layer="16"/>
 </signal>
-<signal name="CVIN4">
+<signal name="MCUADC3">
 <contactref element="R34" pad="2"/>
 <contactref element="IC6" pad="1"/>
@@
 <wire x1="61.656" y1="8.2525" x2="61.6585" y2="8.255" width="0.254" layer="16"/>
 </signal>
-<signal name="CVIN5">
+<signal name="MCUADC2">
 <contactref element="R36" pad="2"/>
 <contactref element="IC6" pad="7"/>
@@
 <via x="6.6675" y="27.7495" extent="1-16" drill="0.6"/>
 </signal>
-<signal name="CVIN6">
+<signal name="MCUADC1">
 <contactref element="POT1" pad="W"/>
 <contactref element="C16" pad="1"/>
