File: main/quantizer_main.sch (EAGLE design)
At the start: 141 parts, among them IC1 TL074D, IC100 REG1117, IC2 TL074D, IC200 REG1117, IC3 TL074D, IC3000 6N138, IC4 TL074D, IC500 MAX6070, IC600 MAX1303_ADC, IC700 MAX5134_DAC, IC800 MKE02_44PIN

Commit message: ewr
Connections:
- net CVIN0: now also TP1.TP
- net CVIN1: now also TP2.TP
- net CVIN2: now also TP3.TP
- net CVIN3: now also TP4.TP
- net CVIN5: now also TP5.TP
- net CVIN6: now also TP6.TP
- net CVIN7: now also TP7.TP
Other:
- note added: "(MAX1303)"
- note added: "(MAX5134)"
- note added: "(MAX6070)"
- note added: "+5V ANALOG"
- note added: "+5V DIGITAL"
- note added: "2 x GAIN BUFFERS"
- note added: "4.096V REF"
- note added: "ADC 16-BIT SPI"
- note added: "ARM M0+ MCU"
- note added: "DAC 16-BIT SPI"
- note added: "GND LINK"
- note added: "MIDI INPUT"
- note added: "MKE02Z64VLD4"
- note added: "POWER INPUT"
- note added: "TRIGGER OUTPUT"
- note added: "VOLTAGE INPUTS FOR ADC"
- note added: "VOLTAGE OUTPUTS"
- moved on the sheet: C1000, C1001, C1200, C1201, C500, C501, C600, C601, C603, C800, C801, C802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

Commit message: sddd
Parts:
- removed TP9: TPB1,27, testpad:TPB1,27
Connections:
- net N$50 renamed OFFSET
- removed net N$46: IC800.PTC2, TP9.TP
- net CVIN6: now also IC800.PTC2
Other:
- note added: "(Used to bring -ve voltage above 0 for MCU ADC ins)"
- note added: "CONTROL POT"
- note added: "HEADERS"
- note added: "OFFSET VOLTAGE BUFFER"
- note added: "VOLTAGE INPUTS FOR 16BIT ADC"
- note added: "VOLTAGE INPUTS FOR MCU ADC"
- note removed: "VOLTAGE INPUTS FOR ADC"
- moved on the sheet: C1400, C1401, C1500, C1700, CVINE, CVINF, IC4A, IC4B, IC4C, R1400, R1401, R1500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

Commit message: sf
Parts:
- removed C1401, C802: (no value), rcl:C-EUC0805
- removed IC600: MAX1303_ADC, jason_eagle6:MAX1303_ADC
- added C29, C30: (no value), rcl:CPOL-EUE2-5
- added IC6: TL074D, linear:TL074D
- C19, C20: device rcl:CPOL-EUE2-5 -> rcl:C-EUC0805
- IC3: value TL074D -> MAX1303_ADC; device linear:TL074D -> jason_eagle6:MAX1303_ADC
- renumbered C100 to C15, C1000 to C12, C1001 to C13, C101 to C14, C102 to C32, C1200 to C8, C1201 to C7, C1400 to C23, C1500 to C22, C1700 to C16, C200 to C35, C2000 to C1, C2001 to C3, C2002 to C5, C201 to C34, C202 to C31, C203 to C33, C2100 to C2, C2200 to C6, C2300 to C4, C2400 to C21, C500 to C27, C501 to C28, C600 to C10, C601 to C9, C603 to C11, C700 to C24, C701 to C26, C702 to C25, C800 to C17, C801 to C18, CVINA to IN2, CVINB to IN1, CVINC to IN5, CVIND to IN4, CVINE to IN3, CVINF to IN6, CVOUTA to OUT4, CVOUTB to OUT3, CVOUTC to OUT1, CVOUTD to OUT2, D3000 to D3, FB1 to L1, FB2 to L2, IC100 to IC9, IC200 to IC10, IC3000 to IC11, IC500 to IC8, IC700 to IC7, IC800 to IC5, JP1 to PWR, JP23 to ICSP, MIDIIN to MIDI, PTC1 to F1, PTC2 to F2, R1000 to R28, R1001 to R26, R1002 to R22, R1003 to R27, R1100 to R25, R1101 to R23, R1102 to R21, R1103 to R24, R1200 to R16, R1201 to R18, R1202 to R20, R1203 to R17, R1300 to R13, R1301 to R15, R1302 to R14, R1303 to R19, R1400 to R33, R1401 to R34, R1500 to R41, R1501 to R40, R1600 to R35, R1601 to R36, R2000 to R1, R2001 to R2, R2002 to R3, R2100 to R4, R2101 to R5, R2102 to R6, R2200 to R12, R2201 to R11, R2202 to R10, R2300 to R9, R2301 to R8, R2302 to R7, R2400 to R39, R2401 to R38, R2402 to R37, R3000 to R29, R3001 to R30, R3002 to R32, R3003 to R31, R3004 to R42, R3005 to R43, R4000 to R44, TP1 to A, TP10 to PD7, TP11 to PD6, TP12 to PD5, TP13 to PB4, TP2 to B, TP3 to C, TP4 to D, TP5 to E, TP6 to F, TP7 to G, TP8 to PB5, TRGOUT to TRIG, U$14 to POT1
Connections:
- removed net CVIN7: C16.1, G.TP, IC5.PTC1, POT1.W
- new net CVIN4: E.TP, IC5.PTC3, IC6A.OUT, R34.2
- net +12V: now also C29.+, IC6P.V+; no longer C19.+, IC3P.V+
- net +5V: now also IC3.AVDD1, IC3.AVDD2, IC3.REFCAP; no longer IC600.AVDD1, IC600.AVDD2, IC600.REFCAP
- net -12V: now also C20.2, C30.-, IC6P.V-; no longer C1401.2, C20.-, IC3P.V-
- net 4.096V: now also IC3.REF; no longer IC600.REF
- net ADC_CSEL: now also IC3.CS#; no longer IC600.CS#
- net ADC_SSTRB: now also IC3.SSTRB; no longer IC600.SSTRB
- net AGND: now also C20.1, C29.-, C30.+, IC3.AGND1, IC3.AGND2, IC3.AGND3, IC4A.+IN, IC4B.+IN, IC4C.+IN, IC4D.+IN; no longer C1401.1, C19.-, C20.+, IC1A.+IN, IC1B.+IN, IC1C.+IN, IC1D.+IN, IC600.AGND1, IC600.AGND2, IC600.AGND3
- net CVIN0: now also IC3.CH1, IC4B.OUT; no longer IC1B.OUT, IC600.CH1
- net CVIN1: now also IC3.CH0, IC4A.OUT; no longer IC1A.OUT, IC600.CH0
- net CVIN2: now also IC3.CH3; no longer IC600.CH3
- net CVIN3: now also IC3.CH2; no longer IC600.CH2
- net CVIN5: now also F.TP, IC5.PTC2, IC6B.OUT, R36.2; no longer E.TP, IC4A.OUT, IC5.PTC3, R34.2
- net CVIN6: now also C16.1, G.TP, IC5.PTC1, POT1.W; no longer F.TP, IC4B.OUT, IC5.PTC2, R36.2
- net CVOUTA: now also IC1A.+IN; no longer IC3A.+IN
- net CVOUTB: now also IC1B.+IN; no longer IC3B.+IN
- net CVOUTC: now also IC1C.+IN; no longer IC3C.+IN
- net CVOUTD: now also IC1D.+IN; no longer IC3D.+IN
- net GND: now also C19.2, IC3.DGND, IC3.DGND0; no longer C802.2, IC600.DGND, IC600.DGND0
- net N$1: now also IC1A.-IN; no longer IC3A.-IN
- net N$11: now also IC1C.-IN; no longer IC3C.-IN
- net N$13: now also IC1C.OUT; no longer IC3C.OUT
- net N$15: now also IC4C.-IN; no longer IC1C.-IN
- net N$16: now also IC1D.-IN; no longer IC3D.-IN
- net N$18: now also IC1D.OUT; no longer IC3D.OUT
- net N$20: now also IC4C.OUT; no longer IC1C.OUT
- net N$21: now also IC4B.-IN; no longer IC1B.-IN
- net N$25: now also IC4D.-IN; no longer IC1D.-IN
- net N$26: now also IC4D.OUT; no longer IC1D.OUT
- net N$27: now also IC4A.-IN; no longer IC1A.-IN
- net N$34: now also IC6D.-IN; no longer IC4D.-IN
- net N$35: now also IC6D.OUT; no longer IC4D.OUT
- net N$4: now also IC1A.OUT; no longer IC3A.OUT
- net N$42: now also IC6C.+IN; no longer IC4C.+IN
- net N$43: now also IC6A.-IN; no longer IC4A.-IN
- net N$47: now also IC6B.-IN; no longer IC4B.-IN
- net N$6: now also IC1B.-IN; no longer IC3B.-IN
- net N$8: now also IC1B.OUT; no longer IC3B.OUT
- net OFFSET: now also IC6A.+IN, IC6B.+IN, IC6C.-IN, IC6C.OUT; no longer IC4A.+IN, IC4B.+IN, IC4C.-IN, IC4C.OUT
- net SPI_CLK: now also IC3.SCLK; no longer IC600.SCLK
- net SPI_MISO: now also IC3.DOUT; no longer IC600.DOUT
- net SPI_MOSI: now also IC3.DIN; no longer IC600.DIN
- net TRGOUT: now also IC6D.+IN; no longer IC4D.+IN
- net VDD: now also C19.1, IC3.DVDD, IC3.DVDD0; no longer C802.1, IC600.DVDD, IC600.DVDD0
Other:
- moved on the sheet: IC1A, IC1B, IC1C, IC1D, IC4A, IC4B, IC4C, IC4D

Commit message: asd
Connections:
- net AGND: now also C16.2, POT1.A
- net GND: no longer C16.2, POT1.A
Changed lines of the file:
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@@
 <part name="SUPPLY31" library="supply2" deviceset="AGND" device=""/>
 <part name="SUPPLY32" library="supply2" deviceset="AGND" device=""/>
-<part name="GND1" library="supply1" deviceset="GND" device=""/>
 <part name="SUPPLY33" library="supply2" deviceset="+5V" device=""/>
 <part name="E" library="testpad" deviceset="TP" device="B1,27"/>
@@
 <part name="G" library="testpad" deviceset="TP" device="B1,27"/>
 <part name="C16" library="rcl" deviceset="C-EU" device="C0805"/>
-<part name="GND2" library="supply1" deviceset="GND" device=""/>
 <part name="SUPPLY34" library="supply2" deviceset="AGND" device=""/>
 <part name="SUPPLY35" library="supply2" deviceset="AGND" device=""/>
@@
 <part name="ICSP" library="pinhead" deviceset="PINHD-1X5" device=""/>
 <part name="PB4" library="testpad" deviceset="TP" device="B1,27"/>
+<part name="SUPPLY63" library="supply2" deviceset="AGND" device=""/>
+<part name="SUPPLY64" library="supply2" deviceset="AGND" device=""/>
 </parts>
 <sheets>
@@
 <instance part="SUPPLY31" gate="G$1" x="-220.98" y="53.34"/>
 <instance part="SUPPLY32" gate="G$1" x="-220.98" y="99.06"/>
-<instance part="GND1" gate="1" x="-256.54" y="-25.4"/>
 <instance part="SUPPLY33" gate="+5V" x="-256.54" y="10.16"/>
 <instance part="E" gate="G$1" x="-144.78" y="114.3"/>
@@
 <instance part="G" gate="G$1" x="-238.76" y="0"/>
 <instance part="C16" gate="G$1" x="-246.38" y="-15.24"/>
-<instance part="GND2" gate="1" x="-246.38" y="-25.4"/>
 <instance part="SUPPLY34" gate="G$1" x="-63.5" y="269.24"/>
 <instance part="SUPPLY35" gate="G$1" x="35.56" y="269.24"/>
@@
 <attribute name="TP_SIGNAL_NAME" x="-54.61" y="24.13" size="1.778" layer="97" rot="R180"/>
 </instance>
+<instance part="SUPPLY63" gate="G$1" x="-256.54" y="-25.4"/>
+<instance part="SUPPLY64" gate="G$1" x="-246.38" y="-25.4"/>
 </instances>
 <busses>
@@
 </net>
 <net name="GND" class="0">
-<segment>
-<pinref part="POT1" gate="G$1" pin="A"/>
-<pinref part="GND1" gate="1" pin="GND"/>
-<wire x1="-256.54" y1="-17.78" x2="-256.54" y2="-22.86" width="0.1524" layer="91"/>
-</segment>
-<segment>
-<pinref part="GND2" gate="1" pin="GND"/>
-<pinref part="C16" gate="G$1" pin="2"/>
-<wire x1="-246.38" y1="-22.86" x2="-246.38" y2="-20.32" width="0.1524" layer="91"/>
-</segment>
 <segment>
 <pinref part="C31" gate="G$1" pin="-"/>
@@
 <pinref part="SUPPLY62" gate="G$1" pin="AGND"/>
 </segment>
-</net>
+<segment>
+<pinref part="POT1" gate="G$1" pin="A"/>
+<wire x1="-256.54" y1="-17.78" x2="-256.54" y2="-22.86" width="0.1524" layer="91"/>
+<pinref part="SUPPLY63" gate="G$1" pin="AGND"/>
+</segment>
+<segment>
+<pinref part="C16" gate="G$1" pin="2"/>
+<wire x1="-246.38" y1="-22.86" x2="-246.38" y2="-20.32" width="0.1524" layer="91"/>
+<pinref part="SUPPLY64" gate="G$1" pin="AGND"/>
+</segment>
+</net>

Commit message: v1 pcb?
Parts:
- added C36: (no value), resistor:C-EUC0805
- added IC12: 24LC_16BT-I/OT, Microchip-24LCxxx:24LC_16BT-I/OT
- added R45, R46: (no value), rcl:R-EU_R0805
Connections:
- net +5V: now also C36.2, IC12.VCC, R45.2, R46.2
- net GND: now also C36.1, IC12.VSS, IC12.WP
- net SCL: now also IC12.SCL, R45.1
- net SDA: now also IC12.SDA, R46.1
Other:
- note added: "EEPROM 8KBIT"
Changed lines of the file:
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@@
 <part name="SUPPLY63" library="supply2" deviceset="AGND" device=""/>
 <part name="SUPPLY64" library="supply2" deviceset="AGND" device=""/>
+<part name="IC12" library="Microchip-24LCxxx" deviceset="24LC_" device="" technology="16BT-I/OT"/>
+<part name="SUPPLY65" library="supply2" deviceset="+5V" device=""/>
+<part name="C36" library="resistor" deviceset="C-EU" device="C0805"/>
+<part name="GND26" library="SparkFun" deviceset="GND" device=""/>
+<part name="R45" library="rcl" deviceset="R-EU_" device="R0805"/>
+<part name="R46" library="rcl" deviceset="R-EU_" device="R0805"/>
+<part name="SUPPLY66" library="supply2" deviceset="+5V" device=""/>
+<part name="SUPPLY67" library="supply2" deviceset="+5V" device=""/>
 </parts>
 <sheets>
@@
 <text x="-269.24" y="-38.1" size="5.08" layer="91">CONTROL POT</text>
 <text x="109.22" y="-22.86" size="5.08" layer="91">HEADERS</text>
+<text x="43.434" y="-34.798" size="3.81" layer="91">EEPROM 8KBIT</text>
 </plain>
 <instances>
@@
 <instance part="SUPPLY63" gate="G$1" x="-256.54" y="-25.4"/>
 <instance part="SUPPLY64" gate="G$1" x="-246.38" y="-25.4"/>
+<instance part="IC12" gate="A" x="45.72" y="-10.16" smashed="yes">
+<attribute name="NAME" x="58.6486" y="-3.2004" size="2.0828" layer="95" ratio="10" rot="SR0"/>
+</instance>
+<instance part="SUPPLY65" gate="+5V" x="35.56" y="-2.54"/>
+<instance part="C36" gate="G$1" x="35.56" y="-15.24" rot="R180"/>
+<instance part="GND26" gate="1" x="35.56" y="-33.02"/>
+<instance part="R45" gate="G$1" x="53.34" y="7.62" rot="R90"/>
+<instance part="R46" gate="G$1" x="71.12" y="7.62" rot="R90"/>
+<instance part="SUPPLY66" gate="+5V" x="53.34" y="17.78"/>
+<instance part="SUPPLY67" gate="+5V" x="71.12" y="17.78"/>
 </instances>
 <busses>
@@
 <wire x1="144.78" y1="360.68" x2="144.78" y2="375.92" width="0.1524" layer="91"/>
 </segment>
+<segment>
+<pinref part="IC12" gate="A" pin="VCC"/>
+<pinref part="SUPPLY65" gate="+5V" pin="+5V"/>
+<wire x1="45.72" y1="-10.16" x2="35.56" y2="-10.16" width="0.1524" layer="91"/>
+<wire x1="35.56" y1="-10.16" x2="35.56" y2="-5.08" width="0.1524" layer="91"/>
+<pinref part="C36" gate="G$1" pin="2"/>
+<junction x="35.56" y="-10.16"/>
+</segment>
+<segment>
+<pinref part="SUPPLY66" gate="+5V" pin="+5V"/>
+<pinref part="R45" gate="G$1" pin="2"/>
+<wire x1="53.34" y1="15.24" x2="53.34" y2="12.7" width="0.1524" layer="91"/>
+</segment>
+<segment>
+<pinref part="SUPPLY67" gate="+5V" pin="+5V"/>
+<pinref part="R46" gate="G$1" pin="2"/>
+<wire x1="71.12" y1="15.24" x2="71.12" y2="12.7" width="0.1524" layer="91"/>
+</segment>
 </net>
 <net name="GND" class="0">
@@
 <pinref part="C11" gate="G$1" pin="2"/>
 <wire x1="2.54" y1="281.94" x2="7.62" y2="281.94" width="0.1524" layer="91"/>
+</segment>
+<segment>
+<pinref part="IC12" gate="A" pin="WP"/>
+<pinref part="GND26" gate="1" pin="GND"/>
+<wire x1="45.72" y1="-17.78" x2="35.56" y2="-17.78" width="0.1524" layer="91"/>
+<wire x1="35.56" y1="-17.78" x2="35.56" y2="-22.86" width="0.1524" layer="91"/>
+<pinref part="IC12" gate="A" pin="VSS"/>
+<wire x1="35.56" y1="-22.86" x2="35.56" y2="-30.48" width="0.1524" layer="91"/>
+<wire x1="45.72" y1="-22.86" x2="35.56" y2="-22.86" width="0.1524" layer="91"/>
+<junction x="35.56" y="-22.86"/>
+<pinref part="C36" gate="G$1" pin="1"/>
+<junction x="35.56" y="-17.78"/>
 </segment>
 </net>
@@
 <label x="2.54" y="78.74" size="1.778" layer="95"/>
 </segment>
+<segment>
+<pinref part="IC12" gate="A" pin="SCL"/>
+<wire x1="45.72" y1="-15.24" x2="43.18" y2="-15.24" width="0.1524" layer="91"/>
+<wire x1="43.18" y1="-15.24" x2="43.18" y2="0" width="0.1524" layer="91"/>
+<label x="40.64" y="10.16" size="1.778" layer="95"/>
+<pinref part="R45" gate="G$1" pin="1"/>
+<wire x1="43.18" y1="0" x2="43.18" y2="10.16" width="0.1524" layer="91"/>
+<wire x1="53.34" y1="2.54" x2="53.34" y2="0" width="0.1524" layer="91"/>
+<wire x1="53.34" y1="0" x2="43.18" y2="0" width="0.1524" layer="91"/>
+<junction x="43.18" y="0"/>
+</segment>
 </net>
 <net name="SDA" class="0">
@@
 <label x="2.54" y="81.28" size="1.778" layer="95"/>
 </segment>
-</net>
+<segment>
+<pinref part="IC12" gate="A" pin="SDA"/>
+<wire x1="81.28" y1="-10.16" x2="83.82" y2="-10.16" width="0.1524" layer="91"/>
+<wire x1="83.82" y1="-10.16" x2="83.82" y2="0" width="0.1524" layer="91"/>
+<label x="81.28" y="10.16" size="1.778" layer="95"/>
+<pinref part="R46" gate="G$1" pin="1"/>
+<wire x1="83.82" y1="0" x2="83.82" y2="10.16" width="0.1524" layer="91"/>
+<wire x1="71.12" y1="2.54" x2="71.12" y2="0" width="0.1524" layer="91"/>
+<wire x1="71.12" y1="0" x2="83.82" y2="0" width="0.1524" layer="91"/>
+<junction x="83.82" y="0"/>
+</segment>
+</net>
