File: main/quantizer_main.sch (EAGLE design)
At the start: 144 parts, among them IC1 TL074D, IC10 REG1117, IC11 6N138, IC12 24LC_16BT-I/OT, IC2 TL074D, IC3 MAX1303_ADC, IC4 TL074D, IC5 MKE02_44PIN, IC6 TL074D, IC7 MAX5134_DAC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

Commit message: c21 10n
Parts:
- C21: value (none) -> 10n
Changed lines of the file:
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@@
 <part name="R39" library="rcl" deviceset="R-EU_" device="R0805"/>
 <part name="SUPPLY47" library="supply2" deviceset="AGND" device=""/>
-<part name="C21" library="rcl" deviceset="C-EU" device="C0805"/>
+<part name="C21" library="rcl" deviceset="C-EU" device="C0805" value="10n"/>
 <part name="SUPPLY45" library="supply2" deviceset="AGND" device=""/>
 <part name="SUPPLY48" library="supply2" deviceset="AGND" device=""/>

Commit message: asd
Parts:
- C1, C2, C4, C6: value (none) -> 200p
- R33, R35: value (none) -> 120k
- R34, R36, R40: value (none) -> 22k
- R41: value (none) -> 100k
Connections:
- net CVIN4 renamed MCUADC3
- net CVIN5 renamed MCUADC2
- net CVIN6 renamed MCUADC1
Other:
- note added: "2.16v"
Changed lines of the file:
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@@
 <part name="R3" library="rcl" deviceset="R-EU_" device="R0805"/>
 <part name="R1" library="rcl" deviceset="R-EU_" device="R0805"/>
-<part name="C1" library="rcl" deviceset="C-EU" device="C0805"/>
+<part name="C1" library="rcl" deviceset="C-EU" device="C0805" value="200p"/>
 <part name="OUT3" library="thonkiconn" deviceset="WQP-PJ301M-12_JACK" device=""/>
 <part name="R5" library="rcl" deviceset="R-EU_" device="R0805"/>
 <part name="R6" library="rcl" deviceset="R-EU_" device="R0805"/>
 <part name="R4" library="rcl" deviceset="R-EU_" device="R0805"/>
-<part name="C2" library="rcl" deviceset="C-EU" device="C0805"/>
+<part name="C2" library="rcl" deviceset="C-EU" device="C0805" value="200p"/>
 <part name="OUT1" library="thonkiconn" deviceset="WQP-PJ301M-12_JACK" device=""/>
 <part name="R11" library="rcl" deviceset="R-EU_" device="R0805"/>
 <part name="R10" library="rcl" deviceset="R-EU_" device="R0805"/>
 <part name="R12" library="rcl" deviceset="R-EU_" device="R0805"/>
-<part name="C6" library="rcl" deviceset="C-EU" device="C0805"/>
+<part name="C6" library="rcl" deviceset="C-EU" device="C0805" value="200p"/>
 <part name="OUT2" library="thonkiconn" deviceset="WQP-PJ301M-12_JACK" device=""/>
 <part name="R8" library="rcl" deviceset="R-EU_" device="R0805"/>
 <part name="R7" library="rcl" deviceset="R-EU_" device="R0805"/>
 <part name="R9" library="rcl" deviceset="R-EU_" device="R0805"/>
-<part name="C4" library="rcl" deviceset="C-EU" device="C0805"/>
+<part name="C4" library="rcl" deviceset="C-EU" device="C0805" value="200p"/>
 <part name="R26" library="rcl" deviceset="R-EU_" device="R0805"/>
 <part name="R27" library="rcl" deviceset="R-EU_" device="R0805"/>
@@
 <part name="POT1" library="jasons_stuff" deviceset="ALPS_POT_SMALL" device=""/>
 <part name="IC6" library="linear" deviceset="TL074" device="D"/>
-<part name="R33" library="rcl" deviceset="R-EU_" device="R0805"/>
-<part name="R40" library="rcl" deviceset="R-EU_" device="R0805"/>
-<part name="R41" library="rcl" deviceset="R-EU_" device="R0805"/>
-<part name="R34" library="rcl" deviceset="R-EU_" device="R0805"/>
+<part name="R33" library="rcl" deviceset="R-EU_" device="R0805" value="120k"/>
+<part name="R40" library="rcl" deviceset="R-EU_" device="R0805" value="22k"/>
+<part name="R41" library="rcl" deviceset="R-EU_" device="R0805" value="100k"/>
+<part name="R34" library="rcl" deviceset="R-EU_" device="R0805" value="22k"/>
 <part name="SUPPLY7" library="supply2" deviceset="+12V" device=""/>
 <part name="SUPPLY8" library="supply2" deviceset="+12V" device=""/>
@@
 <part name="C20" library="rcl" deviceset="C-EU" device="C0805"/>
 <part name="IN6" library="thonkiconn" deviceset="WQP-PJ301M-12_JACK" device=""/>
-<part name="R35" library="rcl" deviceset="R-EU_" device="R0805"/>
-<part name="R36" library="rcl" deviceset="R-EU_" device="R0805"/>
+<part name="R35" library="rcl" deviceset="R-EU_" device="R0805" value="120k"/>
+<part name="R36" library="rcl" deviceset="R-EU_" device="R0805" value="22k"/>
 <part name="C22" library="rcl" deviceset="C-EU" device="C0805"/>
 <part name="SUPPLY10" library="supply2" deviceset="AGND" device=""/>
@@
 <text x="109.22" y="-22.86" size="5.08" layer="91">HEADERS</text>
 <text x="43.434" y="-34.798" size="3.81" layer="91">EEPROM 8KBIT</text>
+<text x="-170.18" y="-11.684" size="1.778" layer="97">2.16v</text>
+<text x="-131.572" y="-12.7" size="1.778" layer="97">2.16v</text>
 </plain>
 <instances>
@@
 </segment>
 </net>
-<net name="CVIN4" class="0">
+<net name="MCUADC3" class="0">
 <segment>
 <pinref part="R34" gate="G$1" pin="2"/>
@@
 </segment>
 </net>
-<net name="CVIN5" class="0">
+<net name="MCUADC2" class="0">
 <segment>
 <pinref part="R36" gate="G$1" pin="2"/>
@@
 </segment>
 </net>
-<net name="CVIN6" class="0">
+<net name="MCUADC1" class="0">
 <segment>
 <pinref part="POT1" gate="G$1" pin="W"/>
